File: PCB PUERTA/PCB PUERTA.kicad_pcb (KiCad board)
At the start: 2 copper layers, 35 parts, among them J1 LIMIT SWITCHES, J2 LLAVE, J3 Screw_Terminal_01x03, J4 Screw_Terminal_01x02, J5 ALIMENTACION, J6 MOTOR, J7 LAMP, K1 FINDER-36.11, K2 FINDER-36.11, Q1 PZT2222A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

Commit message: 13.02.25.8.10
Parts:
- moved J6 103.1 mm to (184.7, 117.7), turned to 90 degrees
- moved K2 79.8 mm to (185.0, 93.0), turned to -90 degrees
- moved K1 79.6 mm to (184.9, 71.8), turned to -90 degrees
- moved C1 77.7 mm to (174.6, 124.3), turned to 180 degrees
- moved R6 47.0 mm to (121.1, 102.5), turned to 180 degrees
- moved R2 44.2 mm to (121.1, 99.9), turned to 180 degrees
- moved J5 37.1 mm to (167.9, 130.6)
- moved BZ1 19.6 mm to (170.5, 116.9), turned to 180 degrees
- moved J7 6.66 mm to (135.0, 130.7)
- moved J4 6.66 mm to (117.3, 130.9)
- moved U1 4.41 mm to (116.3, 115.4)
- moved R1 4.40 mm to (121.0, 89.7)
- moved R10 4.40 mm to (137.9, 92.3)
- moved R3 4.40 mm to (121.0, 97.3)
- moved R4 4.40 mm to (121.1, 105.0)
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Routing:
- net +5V: track 0.00 -> 222.4 mm, vias 0 -> 1
- net MO1: track 0.00 -> 58.0 mm
- net +3.3V: track 0.00 -> 51.1 mm
- net Net-(Q4-C): track 0.00 -> 38.0 mm, vias 0 -> 1
- net Net-(Q1-C): track 0.00 -> 36.8 mm, vias 0 -> 1
- net PP: track 0.00 -> 30.9 mm
- net FTC: track 0.00 -> 30.8 mm
- net Net-(J7-Pin_2): track 0.00 -> 30.2 mm, vias 0 -> 1
- net LSC: track 0.00 -> 26.0 mm
- net Net-(U1-D27): track 0.00 -> 25.4 mm
- net Net-(U1-D14): track 0.00 -> 22.6 mm
- net MO2: track 0.00 -> 20.9 mm
- net KEYA: track 0.00 -> 19.7 mm
- net Net-(U1-D12): track 0.00 -> 18.9 mm
- net BUZZER: track 0.00 -> 18.8 mm
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- added copper zone on B.Cu, net GND
- added copper zone on F.Cu, net GND
Other:
- board outline added: 91.3 x 69.2 mm
