File: PROYECTO PUERTA ESP32-WROOM-32D/PCB PUERTA/PCB PUERTA.kicad_sch (KiCad schematic)
At the start: 35 parts, among them J1 LIMIT SWITCHES, J2 LLAVE, J3 Screw_Terminal_01x03, J4 Screw_Terminal_01x02, J5 ALIMENTACION, J6 MOTOR, J7 LAMP, K1 FINDER-36.11, K2 FINDER-36.11, Q1 PZT2222A, Q2 PZT2222A, Q3 PZT2222A, Q4 PZT2222A, SW1 SW_DIP_x04, U1 ESP32-DEVKITC

Commit message: 20.03.2025
Parts:
- removed J5: ALIMENTACION, TerminalBlock:TerminalBlock_bornier-2_P5.08mm, symbol Connector:Screw_Terminal_01x02
- removed Q1, Q2, Q3, Q4: PZT2222A, Package_TO_SOT_SMD:SOT-223-3_TabPin2, symbol Transistor_BJT:PZT2222A
- removed R12, R13, R14: 1k, Resistor_SMD:R_0402_1005Metric, symbol Device:R_Small_US
- added C2, C3, C4, C5, C6: 100nF, Capacitor_SMD:C_0402_1005Metric, symbol Device:C_Small
- added C7: 22uF, Capacitor_SMD:CP_Elec_5x5.4, symbol Device:C_Polarized_Small
- added D1, D2, D3, D4, D5, D6: ESD9B3.3ST5G, Diode_SMD:D_SOD-923, symbol Diode:ESD9B3.3ST5G
- added D12, D13: MA, LED_SMD:LED_0402_1005Metric, symbol Device:LED
- added D7: 3V3, LED_SMD:LED_0402_1005Metric, symbol Device:LED
- added D8: 5V, LED_SMD:LED_0402_1005Metric, symbol Device:LED
- added D9: 12V, LED_SMD:LED_0402_1005Metric, symbol Device:LED
- added J5: Screw_Terminal_01x04, TerminalBlock:TerminalBlock_bornier-4_P5.08mm, symbol Connector:Screw_Terminal_01x04
- added R15: 100k, Capacitor_SMD:C_0402_1005Metric, symbol Device:R_Small_US
- added R17: 0.1, Resistor_SMD:R_2512_6332Metric, symbol Device:R_Small_US
- added R19, R20, R7, R8, R9: 220, Resistor_SMD:R_0402_1005Metric, symbol Device:R_Small_US
- added U2, U4, U5, U6: MMUN2233LT1G, LIBRERIA PERSONAL:SOT-23-3_1P4X3P040_ONS-L, symbol LIBRERIA PERSONAL:MMUN2233LT1G
- added U3: LM358, LIBRERIA PERSONAL:lm358, symbol Amplifier_Operational:LM358
- BZ1: footprint Buzzer_Beeper:Buzzer_CUI_CPT-9019S-SMT -> Buzzer_Beeper:Buzzer_TDK_PS1240P02BT_D12.2mm_H6.5mm; Part number (none) -> HNB09A05
- C1: value 22u -> 100nF; Part number (none) -> CL05B104KO5NNNC; Voltage (none) -> 16V
- D10: renamed from D1; Part number (none) -> NCD0402R1
- D11: renamed from D2; Part number (none) -> NCD0402R1
- J1: Part number (none) -> YC0321500000G
- J2, J3: Part number (none) -> DB128V-5.08-3P-GN-S
- J4, J6, J7: Part number (none) -> WJ500V-5.08-2P
- R1, R2: Part number (none) -> CRCW04021K00FKED
- R10: renamed from R7; Part number (none) -> CRCW04021K00FKED
- R11: Part number (none) -> CRCW0402220RFKED
- R12: renamed from R8; Part number (none) -> CRCW04021K00FKED
- R13: renamed from R9; Part number (none) -> CRCW04021K00FKED
- R14: renamed from R10; Part number (none) -> CRCW04021K00FKED
- R16: value 1k -> 20k; footprint Resistor_SMD:R_0402_1005Metric -> Capacitor_SMD:C_0402_1005Metric; Part number (none) -> CRCW040220K0FKEDHP
- R18: renamed from R15; Part number (none) -> CRCW0402220RFKED
- R3: renamed from R4; Part number (none) -> CRCW04021K00FKED
- R4: renamed from R3; Part number (none) -> CRCW04021K00FKED
- R5: renamed from R6; Part number (none) -> CRCW04021K00FKED
- R6: renamed from R5; Part number (none) -> CRCW04021K00FKED
- SW1: footprint Button_Switch_SMD:SW_DIP_SPSTx04_Slide_9.78x12.34mm_W8.61mm_P2.54mm -> Button_Switch_SMD:SW_DIP_SPSTx04_Slide_KingTek_DSHP04TS_W7.62mm_P1.27mm; Part number (none) -> DSHP04TSGER
Connections:
- net +3.3V: now also J5.4 (Pin_4), R7.2, U3.8 (V+); no longer U1.1 (3V3)
- net +5V: now also C7.1, J5.3 (Pin_3), R8.2; no longer C1.1, K1.12, K1.A1, K2.12, K2.A1
- net BUZZER: now also R19.2, U4.1 (BASE)
- net FTC: now also C4.1, D4.2 (A2)
- net GND: now also R16.2, C2.2, C3.2, C4.2, C5.2, C6.2, C7.2, D1.1 (A1), D12.1 (K), D13.1 (K), D2.1 (A1), D3.1 (A1), D4.1 (A1), D5.1 (A1), D6.1 (A1), D7.1 (K), D8.1 (K), D9.1 (K), J5.1 (Pin_1), R17.1, U2.2 (EMITTER), U3.4 (V-), U4.2 (EMITTER), U5.2 (EMITTER), U6.2 (EMITTER); no longer K1.14, K2.14
- net KEYA: now also C2.1, D2.2 (A2)
- net KEYC: now also C5.1, D5.2 (A2)
- net LSA: now also C1.1, D1.2 (A2)
- net LSC: now also C6.1, D6.2 (A2)
- net MA: now also U2.1 (BASE)
- net MC: now also U6.1 (BASE); no longer R16.1
- net PP: now also C3.1, D3.2 (A2)
- net at K2.A2: now also U6.3 (COLLECTOR)
- net at BZ1.2 (-): now also U4.3 (COLLECTOR)
- net at J7.2 (Pin_2): now also U5.3 (COLLECTOR)
- net at K1.A2: now also U2.3 (COLLECTOR)
- net at U1.22 (D33): now also R15.1, U3.1
- new net: D8.2 (A), R8.1
- new net: R15.2, R16.1, U3.2 (-)
- new net: D13.2 (A), R20.1
- new net: R20.2, U5.1 (BASE)
- new net: D7.2 (A), R7.1
- new net: D12.2 (A), R19.1
- new net: D9.2 (A), R9.1
- new net +12V: J5.2 (Pin_2), K1.12, K1.A1, K2.12, K2.A1, R9.2
- new net RefCorriente: K1.14, K2.14, R17.2, U3.3 (+)
- no-connect marks 0 -> 3
Other:
- moved on the sheet: BZ1, D10, D11, J1, J2, J3, J4, J6, J7, K1, K2, R1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

Commit message: agregando emulador NE555
Parts:
- added J8: Screw_Terminal_01x02, CONN-TH_P5.08_KF128-5.08-2P, symbol Connector:Screw_Terminal_01x02
Changed lines of the file:
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@@
 (kicad_sch
-	(version 20231120)
+	(version 20250114)
 	(generator "eeschema")
-	(generator_version "8.0")
+	(generator_version "9.0")
 	(paper "A3")
 	(junction
@@
 	)
 	(symbol
+		(lib_id "Connector:Screw_Terminal_01x02")
+		(at 35.56 262.89 180)
+		(unit 1)
+		(exclude_from_sim no)
+		(in_bom yes)
+		(on_board yes)
+		(dnp no)
+		(fields_autoplaced yes)
+		(property "Reference" "J8"
+			(at 35.56 254 0)
+			(effects
+				(font
+					(size 1.27 1.27)
+				)
+			)
+		)
+		(property "Value" "Screw_Terminal_01x02"
+			(at 35.56 256.54 0)
+			(effects
+				(font
+					(size 1.27 1.27)
+				)
+			)
+		)
+		(property "Footprint" "CONN-TH_P5.08_KF128-5.08-2P"
+			(at 35.56 262.89 0)
+			(effects
+				(font
+					(size 1.27 1.27)
+				)
+				(hide yes)
+			)
+		)
+		(property "Datasheet" "~"
+			(at 35.56 262.89 0)
+			(effects
+				(font
+					(size 1.27 1.27)
+				)
+				(hide yes)
+			)
+		)
+		(property "Description" "Generic screw terminal, single row, 01x02, script generated (kicad-library-utils/schlib/autogen/connector/)"
+			(at 35.56 262.89 0)
+			(effects
+				(font
+					(size 1.27 1.27)
+				)
+				(hide yes)
+			)
+		)
+		(property "Part number" "WJ500V-5.08-2P"
+			(at 35.56 262.89 0)
+			(effects
+				(font
+					(size 1.27 1.27)
+				)
+				(hide yes)
+			)
+		)
+		(pin "2"
+		)
+		(pin "1"
+		)
+		(instances
+			(project "PCB PUERTA"
+				(path "/68346520-92d8-4bb7-a413-edc714e7191e"
+					(reference "J8")
+					(unit 1)
+				)
+			)
+		)
+	)
+	(symbol
 		(lib_id "power:+3.3V")
 		(at 73.66 176.53 0)
@@
 		)
 	)
+	(embedded_fonts no)
 )
